File: mother-board/mother.kicad_pcb (KiCad board)
At the start: 2 copper layers, 178.4 x 51.4 mm, 36 parts, among them J1 Screw_Terminal_01x02, J10 Conn_02x03_Odd_Even, J11 Screw_Terminal_01x02, J12 Screw_Terminal_01x02, J2 Screw_Terminal_01x02, J3 Screw_Terminal_01x02, J4 Screw_Terminal_01x02, J5 Screw_Terminal_01x02, J6 Screw_Terminal_01x02, J7 Screw_Terminal_01x02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

Commit message: add rev 0 boards
Parts:
- removed J10: Conn_02x03_Odd_Even, Connector_IDC:IDC-Header_2x03_P2.54mm_Vertical
- added G***: LOGO, SMM:smm-spiral-10mm, F.Cu at (156.7, 85.6)
- added U3: Adafruit_Metro_Mini, SMM:Metro-Mini, F.Cu at (67.8, 98.6)
- moved JP2 30.7 mm to (55.9, 96.8), turned to 90 degrees
- moved U1 26.0 mm to (50.0, 97.3), turned to 90 degrees
- moved JP1 23.3 mm to (50.3, 104.9), turned to 180 degrees
Connections:
- JP1 pad 2: +5V -> +VDC
Routing:
- net GNDPWR: track 242.5 -> 210.0 mm
- net /LATCH: track 173.1 -> 140.6 mm
- net /SERIN: track 83.9 -> 54.1 mm, vias 1 -> 0
- net GNDD: track 194.9 -> 173.5 mm
- net /CLOCK: track 173.4 -> 156.4 mm
- net Net-(JP1-Pad1): track 19.0 -> 34.8 mm
- net +5V: track 325.5 -> 338.2 mm
- net /D0: track 85.2 -> 89.3 mm
- net /D1: track 62.1 -> 63.7 mm
- net +VDC: track 423.7 -> 424.2 mm
Other:
- board text added: "Science Museum of Minnesota Power Shift Register - Mother Board"
